File: header_2x5_2.54_F_RA_to_1.27_M/header_2x5_2.54_F_RA_to_1.27_M.sch (KiCad schematic (older format))
At the start: 2 parts, among them J1 2.54_F_RA, J2 1.27_M

Commit message: Add 'header_2x5_2.54_F_RA_to_1.27_M' adapter board
Parts:
- J2: footprint ng_conn:Samtec_FTSH-105-XX-X-DV -> ng_conn:Samtec_FTSH-105-XX-X-DV-Mating
Changed lines of the file:
@@
 F 0 "J2" H 5900 5167 50  0000 C CNN
 F 1 "1.27_M" H 5900 5076 50  0000 C CNN
-F 2 "ng_conn:Samtec_FTSH-105-XX-X-DV" H 5850 4750 50  0001 C CNN
+F 2 "ng_conn:Samtec_FTSH-105-XX-X-DV-Mating" H 5850 4750 50  0001 C CNN
 F 3 "~" H 5850 4750 50  0001 C CNN
 	1    5850 4750
