File: FT2232H_USB-C_to_2x10_1.27_F_RA/FT2232H_USB-C_to_2x10_1.27_F_RA.kicad_pcb (KiCad board)
At the start: 4 copper layers, 43 x 60 mm, 45 parts, among them J1 USB_C_USB2.0, J2 Conn_02x10_Odd_Even, J3 Conn_02x10_Odd_Even, U1 FT2232HL, U2 93C46BT-I_OT, U3 USBLC6-2SC6, U4 LDO_SOT-23-5, X1 DSC60xx

Commit message: Fix solder mask clearance/minimum width and reexport gerbers
Other:
- rule pad_to_mask_clearance: 0.051 -> 0.05
- rule solder_mask_min_width: 0.25 -> 0.1
